Commit message: files and updated symlink installation manifest.

File: bruno/urdf/bruno.urdf.xacro (robot description, xacro)
@@ -1,3 +1,3 @@
-<?xml version="1.8" ?>
+<?xml version="1.0" ?>
 <robot
   name="bruno" xmlns:xacro="http://ros.org/wiki/xacro">
@@ -100,9 +100,5 @@
     <axis
       xyz="0 0 1" />
-    <limit
-      lower="0"
-      upper="0"
-      effort="0"
-      velocity="0" />
+    <limit lower="-3.14" upper="3.14" effort="1.0" velocity="0.5"/>
   </joint>
   <link
@@ -158,9 +154,5 @@
     <axis
       xyz="0 0 -1" />
-    <limit
-      lower="0"
-      upper="0"
-      effort="0"
-      velocity="0" />
+    <limit lower="-3.14" upper="3.14" effort="0.0" velocity="0.0"/>
   </joint>
   <link
@@ -216,9 +208,5 @@
     <axis
       xyz="0 0 -1" />
-    <limit
-      lower="0"
-      upper="0"
-      effort="0"
-      velocity="0" />
+    <limit lower="-3.14" upper="3.14" effort="1.0" velocity="0.5"/>
   </joint>
   <link
@@ -274,9 +262,5 @@
     <axis
       xyz="0 0 1" />
-    <limit
-      lower="0"
-      upper="0"
-      effort="0"
-      velocity="0" />
+    <limit lower="-3.14" upper="3.14" effort="1.0" velocity="0.5"/>
   </joint>
   <link
@@ -332,9 +316,5 @@
     <axis
       xyz="0 0 -1" />
-    <limit
-      lower="0"
-      upper="0"
-      effort="0"
-      velocity="0" />
+    <limit lower="-3.14" upper="3.14" effort="1.0" velocity="0.5"/>
   </joint>
   <link
@@ -390,9 +370,5 @@
     <axis
       xyz="0 0 1" />
-    <limit
-      lower="0"
-      upper="0"
-      effort="0"
-      velocity="0" />
+    <limit lower="-3.14" upper="3.14" effort="1.0" velocity="0.5"/>
   </joint>
   <link
@@ -448,9 +424,5 @@
     <axis
       xyz="0 0 1" />
-    <limit
-      lower="0"
-      upper="0"
-      effort="0"
-      velocity="0" />
+    <limit lower="-3.14" upper="3.14" effort="1.0" velocity="0.5"/>
   </joint>
   <link
@@ -506,9 +478,5 @@
     <axis
       xyz="0 0 -1" />
-    <limit
-      lower="0"
-      upper="0"
-      effort="0"
-      velocity="0" />
+    <limit lower="-3.14" upper="3.14" effort="1.0" velocity="0.5"/>
   </joint>
   <link
@@ -564,9 +532,5 @@
     <axis
       xyz="0 0 -1" />
-    <limit
-      lower="0"
-      upper="0"
-      effort="0"
-      velocity="0" />
+    <limit lower="-3.14" upper="3.14" effort="1.0" velocity="0.5"/>
   </joint>
   <link
@@ -622,9 +586,5 @@
     <axis
       xyz="0 0 1" />
-    <limit
-      lower="0"
-      upper="0"
-      effort="0"
-      velocity="0" />
+    <limit lower="-3.14" upper="3.14" effort="1.0" velocity="0.5"/>
   </joint>
   <link
@@ -680,9 +640,5 @@
     <axis
       xyz="0 0 -1" />
-    <limit
-      lower="0"
-      upper="0"
-      effort="0"
-      velocity="0" />
+    <limit lower="-3.14" upper="3.14" effort="1.0" velocity="0.5"/>
   </joint>
   <link
@@ -738,9 +694,5 @@
     <axis
       xyz="0 0 1" />
-    <limit
-      lower="0"
-      upper="0"
-      effort="0"
-      velocity="0" />
+    <limit lower="-3.14" upper="3.14" effort="1.0" velocity="0.5"/>
   </joint>
   <link
@@ -939,5 +891,5 @@
   </sensor>
   </gazebo>
-  <!-- <gazebo reference="base_link">
+  <gazebo reference="base_link">
   <gravity>false</gravity>
   <sensor name="imu_sensor" type="imu">
@@ -961,10 +913,10 @@
     <pose>0 0 0 0 0 0</pose>
   </sensor>
-  </gazebo> -->
+  </gazebo>
   <gazebo>
-  <!-- <plugin filename="libodometry_plugin.so" name="odometry_plugin">
+  <plugin filename="libodometry_plugin.so" name="odometry_plugin">
     <frame>base_link</frame>
     <world_frame>fixed_world</world_frame>
-  </plugin> -->
+  </plugin>
   </gazebo>
   <xacro:macro name="body_color">

Commit message: Refactored urdf

File: bruno/urdf/bruno.urdf.xacro (robot description, xacro)
@@ -1,853 +1,903 @@
 <?xml version="1.0" ?>
-<robot
-  name="bruno" xmlns:xacro="http://ros.org/wiki/xacro">
-  <link name="dummy_link"></link>
-  <link
-    name="base_link" >
-    <inertial>
-      <origin
-        xyz="0.0226398495790573 -3.89308433540458E-05 -0.0917853865936327"
-        rpy="0 0 0" />
-      <mass
-        value="40.9811213814977" />
-      <inertia
-        ixx="0.705590024772154"
-        ixy="-0.000426844603876142"
-        ixz="0.0538798871665836"
-        iyy="2.10623867387607"
-        iyz="8.22509666239292E-05"
-        izz="2.66085772664499" />
-    </inertial>
-    <visual>
-      <origin
-        xyz="0 0 0"
-        rpy="0 0 0" />
-      <geometry>
-        <mesh
-          filename="package://bruno/meshes/base_link.STL" />
-      </geometry>
-      <material
-        name="">
-        <color
-          rgba="0.792156862745098 0.819607843137255 0.933333333333333 1" />
-      </material>
-    </visual>
-    <collision>
-      <origin
-        xyz="0 0 0"
-        rpy="0 0 0" />
-      <geometry>
-        <mesh
-          filename="package://bruno/meshes/base_link.STL" />
-      </geometry>
-    </collision>
-  </link>
-  <joint name="dummy_joint" type="fixed">
-    <origin rpy="0 0 0" xyz="0 0 0" />
-    <parent link="dummy_link"/>
-    <child link="base_link"/>
-  </joint>
-  <link
-    name="fr_thigh_link">
-    <inertial>
-      <origin
-        xyz="-0.0632805867054035 2.1285884999056E-09 0.0305615244081003"
-        rpy="0 0 0" />
-      <mass
-        value="2.03276391085227" />
-      <inertia
-        ixx="0.00362430847918608"
-        ixy="-6.93144774285455E-10"
-        ixz="0.000758555151467763"
-        iyy="0.00831656981525165"
-        iyz="2.36222199008423E-10"
-        izz="0.00835118856419136" />
-    </inertial>
-    <visual>
-      <origin
-        xyz="0 0 0"
-        rpy="0 0 0" />
-      <geometry>
-        <mesh
-          filename="package://bruno/meshes/fr_thigh_link.STL" />
-      </geometry>
-      <material
-        name="">
-        <color
-          rgba="0.792156862745098 0.819607843137255 0.933333333333333 1" />
-      </material>
-    </visual>
-    <collision>
-      <origin
-        xyz="0 0 0"
-        rpy="0 0 0" />
-      <geometry>
-        <mesh
-          filename="package://bruno/meshes/fr_thigh_link.STL" />
-      </geometry>
-    </collision>
-  </link>
-  <joint
-    name="fr_thigh_joint"
-    type="revolute">
-    <origin
-      xyz="0.308523286801734 -0.170000173902694 -0.0943774201689784"
-      rpy="1.5707963267949 0 1.5707963267949" />
-    <parent
-      link="base_link" />
-    <child
-      link="fr_thigh_link" />
-    <axis
-      xyz="0 0 1" />
-    <limit lower="-3.14" upper="3.14" effort="1.0" velocity="0.5"/>
-  </joint>
-  <link
-    name="fr_leg_link">
-    <inertial>
-      <origin
-        xyz="0.12019790111426 -0.143259479284328 0.0203781049178077"
-        rpy="0 0 0" />
-      <mass
-        value="2.21745458605018" />
-      <inertia
-        ixx="0.0266716191184848"
-        ixy="0.0187884251532103"
-        ixz="-0.00116911776317338"
-        iyy="0.0200463346888596"
-        iyz="0.00139351727422659"
-        izz="0.0434443595227279" />
-    </inertial>
-    <visual>
-      <origin
-        xyz="0 0 0"
-        rpy="0 0 0" />
-      <geometry>
-        <mesh
-          filename="package://bruno/meshes/fr_leg_link.STL" />
-      </geometry>
-      <material
-        name="">
-        <color
-          rgba="0.792156862745098 0.819607843137255 0.933333333333333 1" />
-      </material>
-    </visual>
-    <collision>
-      <origin
-        xyz="0 0 0"
-        rpy="0 0 0" />
-      <geometry>
-        <mesh
-          filename="package://bruno/meshes/fr_leg_link.STL" />
-      </geometry>
-    </collision>
-  </link>
-  <joint
-    name="fr_leg_joint"
-    type="revolute">
-    <origin
-      xyz="-0.170183232756006 0 0.0354382464541242"
-      rpy="0 1.5707963267949 0" />
-    <parent
-      link="fr_thigh_link" />
-    <child
-      link="fr_leg_link" />
-    <axis
-      xyz="0 0 -1" />
-    <limit lower="-3.14" upper="3.14" effort="0.0" velocity="0.0"/>
-  </joint>
-  <link
-    name="fr_shin_link">
-    <inertial>
-      <origin
-        xyz="0.179968891055547 0.215776713253008 0.000215390278360372"
-        rpy="0 0 0" />
-      <mass
-        value="3.17121221400824" />
-      <inertia
-        ixx="0.0519451453620737"
-        ixy="-0.0399304170181899"
-        ixz="-8.01801154788949E-05"
-        iyy="0.0379833163092041"
-        iyz="-9.46092673541023E-05"
-        izz="0.0858857153551078" />
-    </inertial>
-    <visual>
-      <origin
-        xyz="0 0 0"
-        rpy="0 0 0" />
-      <geometry>
-        <mesh
-          filename="package://bruno/meshes/fr_shin_link.STL" />
-      </geometry>
-      <material
-        name="">
-        <color
-          rgba="0.792156862745098 0.819607843137255 0.933333333333333 1" />
-      </material>
-    </visual>
-    <collision>
-      <origin
-        xyz="0 0 0"
-        rpy="0 0 0" />
-      <geometry>
-        <mesh
-          filename="package://bruno/meshes/fr_shin_link.STL" />
-      </geometry>
-    </collision>
-  </link>
-  <joint
-    name="fr_shin_joint"
-    type="revolute">
-    <origin
-      xyz="0.264190523301229 -0.297986287064543 0.0249999734100426"
-      rpy="0 0 3.14159265358979" />
-    <parent
-      link="fr_leg_link" />
-    <child
-      link="fr_shin_link" />
-    <axis
-      xyz="0 0 -1" />
-    <limit lower="-3.14" upper="3.14" effort="1.0" velocity="0.5"/>
-  </joint>
-  <link
-    name="fl_thigh_link">
-    <inertial>
-      <origin
-        xyz="0.0632805867054036 -2.12868082882789E-09 0.0305615244081003"
-        rpy="0 0 0" />
-      <mass
-        value="2.03276391085227" />
-      <inertia
-        ixx="0.00362430847918608"
-        ixy="-6.93137931212592E-10"
-        ixz="-0.000758555151467763"
-        iyy="0.00831656981525165"
-        iyz="-2.36222192593191E-10"
-        izz="0.00835118856419137" />
-    </inertial>
-    <visual>
-      <origin
-        xyz="0 0 0"
-        rpy="0 0 0" />
-      <geometry>
-        <mesh
-          filename="package://bruno/meshes/fl_thigh_link.STL" />
-      </geometry>
-      <material
-        name="">
-        <color
-          rgba="0.792156862745098 0.819607843137255 0.933333333333333 1" />
-      </material>
-    </visual>
-    <collision>
-      <origin
-        xyz="0 0 0"
-        rpy="0 0 0" />
-      <geometry>
-        <mesh
-          filename="package://bruno/meshes/fl_thigh_link.STL" />
-      </geometry>
-    </collision>
-  </link>
-  <joint
-    name="fl_thigh_joint"
-    type="revolute">
-    <origin
-      xyz="0.308523286801734 0.170000173902694 -0.0943774201689784"
-      rpy="1.5707963267949 0 1.5707963267949" />
-    <parent
-      link="base_link" />
-    <child
-      link="fl_thigh_link" />
-    <axis
-      xyz="0 0 1" />
-    <limit lower="-3.14" upper="3.14" effort="1.0" velocity="0.5"/>
-  </joint>
-  <link
-    name="fl_leg_link">
-    <inertial>
-      <origin
-        xyz="0.120210884605648 0.143248557446126 0.0203781358138403"
-        rpy="0 0 0" />
-      <mass
-        value="2.21746271008323" />
-      <inertia
-        ixx="0.0266721257111891"
-        ixy="-0.0187883416352741"
-        ixz="-0.00116937614015478"
-        iyy="0.0200458538368986"
-        iyz="-0.0013933496117703"
-        izz="0.0434443467625671" />
-    </inertial>
-    <visual>
-      <origin
-        xyz="0 0 0"
-        rpy="0 0 0" />
-      <geometry>
-        <mesh
-          filename="package://bruno/meshes/fl_leg_link.STL" />
-      </geometry>
-      <material
-        name="">
-        <color
-          rgba="0.792156862745098 0.819607843137255 0.933333333333333 1" />
-      </material>
-    </visual>
-    <collision>
-      <origin
-        xyz="0 0 0"
-        rpy="0 0 0" />
-      <geometry>
-        <mesh
-          filename="package://bruno/meshes/fl_leg_link.STL" />
-      </geometry>
-    </collision>
-  </link>
-  <joint
-    name="fl_leg_joint"
-    type="revolute">
-    <origin
-      xyz="0.170183232756006 0 0.0354382464541242"
-      rpy="3.14159265358979 1.5707963267949 0" />
-    <parent
-      link="fl_thigh_link" />
-    <child
-      link="fl_leg_link" />
-    <axis
-      xyz="0 0 -1" />
-    <limit lower="-3.14" upper="3.14" effort="1.0" velocity="0.5"/>
-  </joint>
-  <link
-    name="fl_shin_link">
-    <inertial>
-      <origin
-        xyz="0.179968891055547 -0.215776713253008 -0.000215390278360372"
-        rpy="0 0 0" />
-      <mass
-        value="3.17121221400824" />
-      <inertia
-        ixx="0.0519451453620737"
-        ixy="0.0399304170181898"
-        ixz="8.01801154788981E-05"
-        iyy="0.0379833163092041"
-        iyz="-9.46092673541049E-05"
-        izz="0.0858857153551077" />
-    </inertial>
-    <visual>
-      <origin
-        xyz="0 0 0"
-        rpy="0 0 0" />
-      <geometry>
-        <mesh
-          filename="package://bruno/meshes/fl_shin_link.STL" />
-      </geometry>
-      <material
-        name="">
-        <color
-          rgba="0.792156862745098 0.819607843137255 0.933333333333333 1" />
-      </material>
-    </visual>
-    <collision>
-      <origin
-        xyz="0 0 0"
-        rpy="0 0 0" />
-      <geometry>
-        <mesh
-          filename="package://bruno/meshes/fl_shin_link.STL" />
-      </geometry>
-    </collision>
-  </link>
-  <joint
-    name="fl_shin_joint"
-    type="revolute">
-    <origin
-      xyz="0.264190523301229 0.297986287064544 0.0250000265899572"
-      rpy="0 0 3.14159265358979" />
-    <parent
-      link="fl_leg_link" />
-    <child
-      link="fl_shin_link" />
-    <axis
-      xyz="0 0 1" />
-    <limit lower="-3.14" upper="3.14" effort="1.0" velocity="0.5"/>
-  </joint>
-  <link
-    name="br_thigh_link">
-    <inertial>
-      <origin
-        xyz="-0.0632805867054036 2.12858870807242E-09 0.0305615244081001"
-        rpy="0 0 0" />
-      <mass
-        value="2.03276391085227" />
-      <inertia
-        ixx="0.00362430847918608"
-        ixy="-6.93144759042335E-10"
-        ixz="0.000758555151467761"
-        iyy="0.00831656981525165"
-        iyz="2.36222195879922E-10"
-        izz="0.00835118856419136" />
-    </inertial>
-    <visual>
-      <origin
-        xyz="0 0 0"
-        rpy="0 0 0" />
-      <geometry>
-        <mesh
-          filename="package://bruno/meshes/br_thigh_link.STL" />
-      </geometry>
-      <material
-        name="">
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
File: install/bruno/share/bruno/urdf/bruno.urdf.xacro (robot description, xacro)
@@ -1 +1 @@
-/home/azif/projetcs/Quadruped-Robot-Performing-SLAM/bruno/urdf/bruno.urdf.xacro
+/home/azif/projects/Quadruped-Robot-Performing-SLAM/bruno/urdf/bruno.urdf.xacro
